Commit message: Add collisions and inetrials to URDF | Initial setup of Gazebo

File: franka_description/robots/hand.xacro (robot description, xacro)
@@ -52,7 +52,18 @@
         </geometry>
       </collision>
+      <inertial>
+        <origin rpy="0 0 0" xyz="-0.01 0 0.03"/>
+        <mass value="0.73"/>
+        <inertia ixx="0.001" ixy="0" ixz="0" iyy="0.0025" iyz="0" izz="0.0017"/>
+      </inertial>
     </link>
     <!-- Define the hand_tcp frame -->
-    <link name="${ns}_hand_tcp"/>
+    <link name="${ns}_hand_tcp">
+      <inertial>
+        <mass value="0"/>
+        <origin rpy="0 0 0" xyz="0 0 0"/>
+        <inertia ixx="0" ixy="0" ixz="0" iyy="0" iyz="0" izz="0"/>
+      </inertial>
+    </link>
     <joint name="${ns}_hand_tcp_joint" type="fixed">
       <origin xyz="0 0 0.1034" rpy="0 0 0"/>
@@ -66,4 +77,37 @@
         </geometry>
       </visual>
+      <!-- screw mount -->
+      <collision>
+        <origin rpy="0 0 0" xyz="0 18.5e-3 11e-3"/>
+        <geometry>
+            <box size="22e-3 15e-3 20e-3"/>
+        </geometry>
+      </collision>
+      <!-- cartriage sledge -->
+      <collision>
+          <origin rpy="0 0 0" xyz="0 6.8e-3 2.2e-3"/>
+          <geometry>
+              <box size="22e-3 8.8e-3 3.8e-3"/>
+          </geometry>
+      </collision>
+      <!-- diagonal finger -->
+      <collision>
+          <origin rpy="0.5235987755982988 0 0" xyz="0 15.9e-3 28.35e-3"/>
+          <geometry>
+              <box size="17.5e-3 7e-3 23.5e-3"/>
+          </geometry>
+      </collision>
+      <!-- rubber tip with which to grasp -->
+      <collision>
+          <origin rpy="0 0 0" xyz="0 7.58e-3 45.25e-3"/>
+          <geometry>
+              <box size="17.5e-3 15.2e-3 18.5e-3"/>
+          </geometry>
+      </collision>
+      <inertial>
+        <origin rpy="0 0 0" xyz="0 0 0"/>
+        <mass value="0.015"/>
+        <inertia ixx="2.3749999999999997e-06" ixy="0" ixz="0" iyy="2.3749999999999997e-06" iyz="0" izz="7.5e-07"/>
+      </inertial>
     </link>
     <link name="${ns}_rightfinger">
@@ -74,4 +118,37 @@
         </geometry>
       </visual>
+      <!-- screw mount -->
+      <collision>
+        <origin rpy="0 0 0" xyz="0 -18.5e-3 11e-3"/>
+        <geometry>
+            <box size="22e-3 15e-3 20e-3"/>
+        </geometry>
+      </collision>
+      <!-- cartriage sledge -->
+      <collision>
+          <origin rpy="0 0 0" xyz="0 -6.8e-3 2.2e-3"/>
+          <geometry>
+              <box size="22e-3 8.8e-3 3.8e-3"/>
+          </geometry>
+      </collision>
+      <!-- diagonal finger -->
+      <collision>
+          <origin rpy="-0.5235987755982988 0 0" xyz="0 -15.9e-3 28.35e-3"/>
+          <geometry>
+              <box size="17.5e-3 7e-3 23.5e-3"/>
+          </geometry>
+      </collision>
+      <!-- rubber tip with which to grasp -->
+      <collision>
+          <origin rpy="0 0 0" xyz="0 -7.58e-3 45.25e-3"/>
+          <geometry>
+              <box size="17.5e-3 15.2e-3 18.5e-3"/>
+          </geometry>
+      </collision>
+      <inertial>
+          <origin rpy="0 0 0" xyz="0 0 0"/>
+          <mass value="0.015"/>
+          <inertia ixx="2.3749999999999997e-06" ixy="0" ixz="0" iyy="2.3749999999999997e-06" iyz="0" izz="7.5e-07"/>
+      </inertial>
     </link>
     <joint name="${ns}_finger_joint1" type="prismatic">

File: franka_description/robots/panda_arm.ros2_control.xacro (robot description, xacro)
@@ -1,15 +1,20 @@
 <?xml version="1.0"?>
 <robot xmlns:xacro="http://www.ros.org/wiki/xacro">
-  <xacro:macro name="panda_arm_ros2_control" params="ns robot_ip use_fake_hardware:=^|false fake_sensor_commands:=^|false">
+  <xacro:macro name="panda_arm_ros2_control" params="ns robot_ip use_fake_hardware:=^|false fake_sensor_commands:=^|false use_sim:=^|false parameters_file:=^|''">
     <ros2_control name="FrankaHardwareInterface" type="system">
       <hardware>
-        <xacro:if value="${use_fake_hardware}">
-          <plugin>fake_components/GenericSystem</plugin>
-          <param name="fake_sensor_commands">${fake_sensor_commands}</param>
-          <param name="state_following_offset">0.0</param>
+        <xacro:if value="${use_sim}">
+          <plugin>ign_ros2_control/IgnitionSystem</plugin>
         </xacro:if>
-        <xacro:unless value="${use_fake_hardware}">
-          <plugin>franka_hardware/FrankaHardwareInterface</plugin>
-          <param name="robot_ip">${robot_ip}</param>
+        <xacro:unless value="${use_sim}">
+          <xacro:if value="${use_fake_hardware}">
+            <plugin>fake_components/GenericSystem</plugin>
+            <param name="fake_sensor_commands">${fake_sensor_commands}</param>
+            <param name="state_following_offset">0.0</param>
+          </xacro:if>
+          <xacro:unless value="${use_fake_hardware}">
+            <plugin>franka_hardware/FrankaHardwareInterface</plugin>
+            <param name="robot_ip">${robot_ip}</param>
+          </xacro:unless>
         </xacro:unless>
       </hardware>
@@ -33,4 +38,12 @@
       <xacro:configure_joint joint_name="${ns}_joint7" initial_position="${pi/4}"/>
     </ros2_control>
+    <xacro:if value="${use_sim}">
+      <gazebo>
+        <plugin filename="ign_ros2_control-system"
+          name="ign_ros2_control::IgnitionROS2ControlPlugin">
+          <parameters>${parameters_file}</parameters>
+        </plugin>
+      </gazebo>
+    </xacro:if>
   </xacro:macro>
 </robot>

File: franka_description/robots/panda_arm.urdf.xacro (robot description, xacro)
@@ -6,6 +6,10 @@
   <xacro:arg name="use_fake_hardware" default="false"/>
   <xacro:arg name="fake_sensor_commands" default="false"/>
+  <xacro:arg name="gazebo" default="false"/>
+  <xacro:arg name="parameters_file" default="$(find franka_bringup)/config/controllers.yaml"/>
+  <xacro:arg name="parent" default="world"/>
   <xacro:include filename="$(find franka_description)/robots/panda_arm.xacro"/>
-  <xacro:panda_arm arm_id="$(arg arm_id)" safety_distance="0.03"/>
+  <xacro:panda_arm arm_id="$(arg arm_id)" safety_distance="0.03" connected_to="$(arg parent)"/>
+  <link name="world" />
   <xacro:if value="$(arg hand)">
     <xacro:include filename="$(find franka_description)/robots/hand.xacro"/>
@@ -13,4 +17,6 @@
   </xacro:if>
   <xacro:include filename="$(find franka_description)/robots/panda_arm.ros2_control.xacro"/>
-  <xacro:panda_arm_ros2_control ns="$(arg arm_id)" robot_ip="$(arg robot_ip)" use_fake_hardware="$(arg use_fake_hardware)" fake_sensor_commands="$(arg fake_sensor_commands)"/>
+  <xacro:panda_arm_ros2_control ns="$(arg arm_id)" robot_ip="$(arg robot_ip)"
+         use_fake_hardware="$(arg use_fake_hardware)" fake_sensor_commands="$(arg fake_sensor_commands)"
+         use_sim="$(arg gazebo)" parameters_file="$(arg parameters_file)"/>
 </robot>

File: franka_description/robots/panda_arm.xacro (robot description, xacro)
@@ -35,4 +35,9 @@
         </geometry>
       </collision>
+      <inertial>
+        <origin rpy="0 0 0" xyz="-0.041018 -0.00014 0.049974"/>
+        <mass value="0.629769"/>
+        <inertia ixx="0.00315" ixy="8.2904e-07" ixz="0.00015" iyy="0.00388" iyz="8.2299e-06" izz="0.004285"/>
+      </inertial>
     </link>
     <link name="${arm_id}_link1">
@@ -60,4 +65,9 @@
         </geometry>
       </collision>
+      <inertial>
+        <origin rpy="0 0 0" xyz="0.003875 0.002081 -0.04762"/>
+        <mass value="4.970684"/>
+        <inertia ixx="0.70337" ixy="-0.000139" ixz="0.006772" iyy="0.70661" iyz="0.019169" izz="0.009117"/>
+      </inertial>
     </link>
     <joint name="${arm_id}_joint1" type="revolute">
@@ -93,4 +103,9 @@
         </geometry>
       </collision>
+      <inertial>
+        <origin rpy="0 0 0" xyz="-0.003141 -0.02872  0.003495"/>
+        <mass value="0.646926"/>
+        <inertia ixx="0.007962" ixy="-0.003925" ixz="0.010254" iyy="0.02811" iyz="0.000704" izz="0.025995"/>
+      </inertial>
     </link>
     <joint name="${arm_id}_joint2" type="revolute">
@@ -126,4 +141,9 @@
         </geometry>
       </collision>
+      <inertial>
+        <origin rpy="0 0 0" xyz="2.7518e-02 3.9252e-02 -6.6502e-02"/>
+        <mass value="3.228604"/>
+        <inertia ixx="0.037242" ixy="-0.004761" ixz="-0.011396" iyy="0.036155" iyz="-0.012805" izz="0.01083"/>
+      </inertial>
     </link>
     <joint name="${arm_id}_joint3" type="revolute">
@@ -159,4 +179,9 @@
         </geometry>
       </collision>
+      <inertial>
+        <origin rpy="0 0 0" xyz="-5.317e-02 1.04419e-01 2.7454e-02"/>
+        <mass value="3.587895"/>
+        <inertia ixx="0.025853" ixy="0.007796" ixz="-0.001332" iyy="0.019552" iyz="0.008641" izz="0.028323"/>
+      </inertial>
     </link>
     <joint name="${arm_id}_joint4" type="revolute">
@@ -210,4 +235,9 @@
         </geometry>
       </collision>
+      <inertial>
+        <origin rpy="0 0 0" xyz="-1.1953e-02 4.1065e-02 -3.8437e-02"/>
+        <mass value="1.225946"/>
+        <inertia ixx="0.035549" ixy="-0.002117" ixz="-0.004037" iyy="0.029474" iyz="0.000229" izz="0.008627"/>
+      </inertial>
     </link>
     <joint name="${arm_id}_joint5" type="revolute">
@@ -243,4 +273,9 @@
         </geometry>
       </collision>
+      <inertial>
+        <origin rpy="0 0 0" xyz="6.0149e-02 -1.4117e-02 -1.0517e-02"/>
+        <mass value="1.666555"/>
+        <inertia ixx="0.001964" ixy="0.000109" ixz="-0.001158" iyy="0.004354" iyz="0.000341" izz="0.005433"/>
+      </inertial>
     </link>
     <joint name="${arm_id}_joint6" type="revolute">
@@ -276,4 +311,9 @@
         </geometry>
       </collision>
+      <inertial>
+        <origin rpy="0 0 0" xyz="1.0517e-02 -4.252e-03 6.1597e-02"/>
+        <mass value="0.735522"/>
+        <inertia ixx="0.012516" ixy="-0.000428" ixz="-0.001196" iyy="0.010027" iyz="-0.000741" izz="0.004815"/>
+      </inertial>
     </link>
     <joint name="${arm_id}_joint7" type="revolute">
@@ -304,4 +344,9 @@
         </geometry>
       </collision>
+      <inertial>
+        <mass value="0"/>
+        <origin rpy="0 0 0" xyz="0 0 0"/>
+        <inertia ixx="0" ixy="0" ixz="0" iyy="0" iyz="0" izz="0"/>
+      </inertial>
     </link>
     <joint name="${arm_id}_joint8" type="fixed">
