Commit message: Add joint params | remove unstable plugin

File: franka_description/robots/panda_arm.ros2_control.xacro (robot description, xacro)
@@ -45,8 +45,4 @@
           <parameters>${parameters_file}</parameters>
         </plugin>
-        <plugin filename="franka_gazebo-plugin"
-          name="franka_gazebo::PandaAntiGravityPlugin">
-          <root_link>${ns}_link0</root_link>
-        </plugin>
       </gazebo>
     </xacro:if>

File: franka_description/robots/panda_arm.xacro (robot description, xacro)
@@ -78,4 +78,5 @@
       <axis xyz="0 0 1"/>
       <limit effort="87" lower="-2.8973" upper="2.8973" velocity="2.1750"/>
+      <dynamics damping="0.0" friction="0.0"/>
     </joint>
     <link name="${arm_id}_link2">
@@ -116,4 +117,5 @@
       <axis xyz="0 0 1"/>
       <limit effort="87" lower="-1.7628" upper="1.7628" velocity="2.1750"/>
+      <dynamics damping="0.0" friction="0.0"/>
     </joint>
     <link name="${arm_id}_link3">
@@ -154,4 +156,5 @@
       <axis xyz="0 0 1"/>
       <limit effort="87" lower="-2.8973" upper="2.8973" velocity="2.1750"/>
+      <dynamics damping="0.0" friction="0.0"/>
     </joint>
     <link name="${arm_id}_link4">
@@ -192,4 +195,5 @@
       <axis xyz="0 0 1"/>
       <limit effort="87" lower="-3.0718" upper="-0.0698" velocity="2.1750"/>
+      <dynamics damping="0.0" friction="0.0"/>
     </joint>
     <link name="${arm_id}_link5">
@@ -248,4 +252,5 @@
       <axis xyz="0 0 1"/>
       <limit effort="12" lower="-2.8973" upper="2.8973" velocity="2.6100"/>
+      <dynamics damping="0.0" friction="0.0"/>
     </joint>
     <link name="${arm_id}_link6">
@@ -286,4 +291,5 @@
       <axis xyz="0 0 1"/>
       <limit effort="12" lower="-0.0175" upper="3.7525" velocity="2.6100"/>
+      <dynamics damping="0.0" friction="0.0"/>
     </joint>
     <link name="${arm_id}_link7">
@@ -324,4 +330,5 @@
       <axis xyz="0 0 1"/>
       <limit effort="12" lower="-2.8973" upper="2.8973" velocity="2.6100"/>
+      <dynamics damping="0.0" friction="0.0"/>
     </joint>
     <link name="${arm_id}_link8">
